Commit message: model test

File: tests/dyros_tocabi_fixed_hand.urdf (robot description, URDF)
Before this commit: robot dyros_tocabi_description, 35 links, 34 joints
Links:
- added link Head_Link, mass 2.006332; collision cylinder length=0.043 radius=0.07; visual mesh filename=package://tocabi_description/meshes/head.STL
- link Neck_Link: mass 2.254332 -> 0.248
Joints:
- added joint Head_Joint: type revolute, parent Neck_Link, child Head_Link, origin xyz=0.0 0.0 0.0275 rpy=0 0 0, axis 0 1 0, limit lower=-1.54 upper=1.54 effort=500 velocity=100
- joint R_Wrist2_Joint: axis 0 -1 0 -> (none); limit lower=-2.094 upper=2.094 effort=500 velocity=100 -> (none); type revolute -> fixed

File: tests/dyros_tocabi_fixed_head2.urdf (robot description, URDF)
Before this commit: robot dyros_tocabi_description, 35 links, 34 joints
Links:
- added link Head_Link, mass 2.006332; collision cylinder length=0.043 radius=0.07; visual mesh filename=package://tocabi_description/meshes/head.STL
- link Neck_Link: mass 2.254332 -> 0.248
Joints:
- added joint Head_Joint: type fixed, parent Neck_Link, child Head_Link, origin xyz=0.0 0.0 0.0275 rpy=0 0 0, limit lower=-1.54 upper=1.54 effort=500 velocity=100
- joint Neck_Joint: axis 0 0 1 -> (none); limit lower=-1.54 upper=1.54 effort=500 velocity=100 -> (none); type revolute -> fixed

File: tests/dyros_tocabi_no_right_arm.urdf (robot description, URDF)
Before this commit: robot dyros_tocabi_description, 35 links, 34 joints
Links:
- added link Head_Link, mass 2.006332; collision cylinder length=0.043 radius=0.07; visual mesh filename=package://tocabi_description/meshes/head.STL
- link Neck_Link: mass 2.254332 -> 0.248
Joints:
- added joint Head_Joint: type revolute, parent Neck_Link, child Head_Link, origin xyz=0.0 0.0 0.0275 rpy=0 0 0, axis 0 1 0, limit lower=-1.54 upper=1.54 effort=500 velocity=100
- joint R_Elbow_Joint: axis 1 0 0 -> (none); limit lower=-2.967 upper=3.14159 effort=500 velocity=100 -> (none); type revolute -> fixed
- joint R_Forearm_Joint: axis 0 -1 0 -> (none); limit lower=-3.14159 upper=3.14159 effort=500 velocity=100 -> (none); type revolute -> fixed
- joint R_Wrist1_Joint: axis 1 0 0 -> (none); limit lower=-3.14159 upper=3.14159 effort=500 velocity=100 -> (none); type revolute -> fixed
- joint R_Wrist2_Joint: axis 0 -1 0 -> (none); limit lower=-2.094 upper=2.094 effort=500 velocity=100 -> (none); type revolute -> fixed

File: tests/dyros_tocabi_no_waist.urdf (robot description, URDF)
Before this commit: robot dyros_tocabi_description, 35 links, 34 joints
Links:
- added link Head_Link, mass 2.006332; collision cylinder length=0.043 radius=0.07; visual mesh filename=package://tocabi_description/meshes/head.STL
- link Neck_Link: mass 2.254332 -> 0.248
Joints:
- added joint Head_Joint: type fixed, parent Neck_Link, child Head_Link, origin xyz=0.0 0.0 0.0275 rpy=0 0 0, axis 0 1 0, limit lower=-1.54 upper=1.54 effort=500 velocity=100
- joint L_Armlink_Joint: type revolute -> fixed
- joint L_Elbow_Joint: type revolute -> fixed
- joint L_Forearm_Joint: type revolute -> fixed
- joint L_Shoulder1_Joint: type revolute -> fixed
- joint L_Shoulder2_Joint: type revolute -> fixed
- joint L_Shoulder3_Joint: type revolute -> fixed
- joint L_Wrist1_Joint: type revolute -> fixed
- joint L_Wrist2_Joint: type revolute -> fixed
- joint Neck_Joint: type revolute -> fixed
- joint R_Armlink_Joint: type revolute -> fixed
- joint R_Elbow_Joint: axis 1 0 0 -> (none); limit lower=-2.967 upper=3.14159 effort=500 velocity=100 -> (none); type revolute -> fixed
- joint R_Forearm_Joint: axis 0 -1 0 -> (none); limit lower=-3.14159 upper=3.14159 effort=500 velocity=100 -> (none); type revolute -> fixed
- joint R_Shoulder1_Joint: type revolute -> fixed
- joint R_Shoulder2_Joint: type revolute -> fixed
- joint R_Shoulder3_Joint: type revolute -> fixed
- joint R_Wrist1_Joint: axis 1 0 0 -> (none); limit lower=-3.14159 upper=3.14159 effort=500 velocity=100 -> (none); type revolute -> fixed
- joint R_Wrist2_Joint: axis 0 -1 0 -> (none); limit lower=-2.094 upper=2.094 effort=500 velocity=100 -> (none); type revolute -> fixed
- joint Upperbody_Joint: type revolute -> fixed
- joint Waist1_Joint: type revolute -> fixed
- joint Waist2_Joint: type revolute -> fixed

File: tests/dyros_tocabi_ub.urdf (robot description, URDF)
Before this commit: robot dyros_tocabi_description, 35 links, 34 joints
Links:
- removed link L_AnkleCenter_Link
- removed link L_AnkleRoll_Link
- removed link L_Foot_Link
- removed link L_HipCenter_Link
- removed link L_HipRoll_Link
- removed link L_Knee_Link
- removed link L_Thigh_Link
- removed link R_AnkleCenter_Link
- removed link R_AnkleRoll_Link
- removed link R_Foot_Link
- removed link R_HipCenter_Link
- removed link R_HipRoll_Link
- removed link R_Knee_Link
- removed link R_Thigh_Link
- added link Head_Link, mass 2.006332; collision cylinder length=0.043 radius=0.07; visual mesh filename=package://tocabi_description/meshes/head.STL
- link Neck_Link: mass 2.254332 -> 0.248
Joints:
- removed joint L_AnklePitch_Joint
- removed joint L_AnkleRoll_Joint
- removed joint L_Foot_Joint
- removed joint L_HipPitch_Joint
- removed joint L_HipRoll_Joint
- removed joint L_HipYaw_Joint
- removed joint L_Knee_Joint
- removed joint R_AnklePitch_Joint
- removed joint R_AnkleRoll_Joint
- removed joint R_Foot_Joint
- removed joint R_HipPitch_Joint
- removed joint R_HipRoll_Joint
- removed joint R_HipYaw_Joint
- removed joint R_Knee_Joint
- added joint Head_Joint: type revolute, parent Neck_Link, child Head_Link, origin xyz=0.0 0.0 0.0275 rpy=0 0 0, axis 0 1 0, limit lower=-1.54 upper=1.54 effort=500 velocity=100

File: tests/dyros_tocabi_upper_body.urdf (robot description, URDF)
Before this commit: robot dyros_tocabi_description, 35 links, 34 joints
Links:
- removed link L_AnkleCenter_Link
- removed link L_AnkleRoll_Link
- removed link L_Foot_Link
- removed link L_HipCenter_Link
- removed link L_HipRoll_Link
- removed link L_Knee_Link
- removed link L_Thigh_Link
- removed link R_AnkleCenter_Link
- removed link R_AnkleRoll_Link
- removed link R_Foot_Link
- removed link R_HipCenter_Link
- removed link R_HipRoll_Link
- removed link R_Knee_Link
- removed link R_Thigh_Link
- added link Head_Link, mass 2.006332; collision cylinder length=0.043 radius=0.07; visual mesh filename=package://tocabi_description/meshes/head.STL
- link Neck_Link: mass 2.254332 -> 0.248
Joints:
- removed joint L_AnklePitch_Joint
- removed joint L_AnkleRoll_Joint
- removed joint L_Foot_Joint
- removed joint L_HipPitch_Joint
- removed joint L_HipRoll_Joint
- removed joint L_HipYaw_Joint
- removed joint L_Knee_Joint
- removed joint R_AnklePitch_Joint
- removed joint R_AnkleRoll_Joint
- removed joint R_Foot_Joint
- removed joint R_HipPitch_Joint
- removed joint R_HipRoll_Joint
- removed joint R_HipYaw_Joint
- removed joint R_Knee_Joint
- added joint Head_Joint: type fixed, parent Neck_Link, child Head_Link, origin xyz=0.0 0.0 0.0275 rpy=0 0 0, axis 0 1 0, limit lower=-1.54 upper=1.54 effort=500 velocity=100
- joint L_Armlink_Joint: type revolute -> fixed
- joint L_Elbow_Joint: type revolute -> fixed
- joint L_Forearm_Joint: type revolute -> fixed
- joint L_Shoulder1_Joint: type revolute -> fixed
- joint L_Shoulder2_Joint: type revolute -> fixed
- joint L_Shoulder3_Joint: type revolute -> fixed
- joint L_Wrist1_Joint: type revolute -> fixed
- joint L_Wrist2_Joint: type revolute -> fixed
- joint Neck_Joint: type revolute -> fixed
- joint R_Armlink_Joint: type revolute -> fixed
- joint R_Elbow_Joint: axis 1 0 0 -> (none); limit lower=-2.967 upper=3.14159 effort=500 velocity=100 -> (none); type revolute -> fixed
- joint R_Forearm_Joint: axis 0 -1 0 -> (none); limit lower=-3.14159 upper=3.14159 effort=500 velocity=100 -> (none); type revolute -> fixed
- joint R_Shoulder1_Joint: type revolute -> fixed
- joint R_Shoulder2_Joint: type revolute -> fixed
- joint R_Shoulder3_Joint: type revolute -> fixed
- joint R_Wrist1_Joint: axis 1 0 0 -> (none); limit lower=-3.14159 upper=3.14159 effort=500 velocity=100 -> (none); type revolute -> fixed
- joint R_Wrist2_Joint: axis 0 -1 0 -> (none); limit lower=-2.094 upper=2.094 effort=500 velocity=100 -> (none); type revolute -> fixed
- joint Upperbody_Joint: type revolute -> fixed
- joint Waist1_Joint: type revolute -> fixed
- joint Waist2_Joint: type revolute -> fixed
